File: Hardware/Pcb/coil_winding_v1/coil_winding_step.kicad_sch (KiCad schematic)
At the start: 25 parts, among them J1 Conn_01x14_Pin, J2 Screw_Terminal_01x02, J3 Conn_01x03_Socket, J4 Conn_01x03_Socket, M1 Motor_DC, Q3 IRFZ40, SW1 SW_SPST, SW2 SW_SPST, SW3 RotaryEncoder_Switch, U1 LM7805_TO220

Commit message: tuesday
Parts:
- removed J4: Conn_01x03_Socket, Connector_PinHeader_2.54mm:PinHeader_1x03_P2.54mm_Vertical, symbol Connector:Conn_01x03_Socket
- added J5: Conn_01x04_Socket, Connector_PinHeader_2.54mm:PinHeader_1x04_P2.54mm_Vertical, symbol Connector:Conn_01x04_Socket
Connections:
- net +5V: now also J5.1 (Pin_1); no longer A1.30 (VIN)
- net D6: now also J5.3 (Pin_3)
- net GND: now also J5.2 (Pin_2)
- net A0: now reaches A1.19 (A0)
- net A0: now also J5.4 (Pin_4)
- no-connect marks 14 -> 15
Changed lines of the file:
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@@
 	)
 	(no_connect
-		(at 143.51 128.27)
+		(at 49.53 152.4)
 	)
 	(no_connect
-		(at 49.53 152.4)
+		(at 128.27 102.87)
 	)
 	(no_connect
@@
 	)
 	(no_connect
+		(at 143.51 130.81)
+	)
+	(no_connect
 		(at 52.07 152.4)
 	)
@@
 	(wire
 		(pts
-			(xy 143.51 138.43) (xy 146.05 138.43)
+			(xy 213.36 153.67) (xy 199.39 153.67)
 		)
 		(stroke
@@
 	(wire
 		(pts
-			(xy 186.69 139.7) (xy 189.23 139.7)
+			(xy 203.2 146.05) (xy 203.2 144.78)
 		)
 		(stroke
@@
 	(wire
 		(pts
-			(xy 189.23 143.51) (xy 189.23 139.7)
+			(xy 143.51 138.43) (xy 146.05 138.43)
 		)
 		(stroke
@@
 	(wire
 		(pts
-			(xy 175.26 55.88) (xy 177.8 55.88)
+			(xy 186.69 139.7) (xy 189.23 139.7)
 		)
 		(stroke
@@
 	(wire
 		(pts
-			(xy 50.8 106.68) (xy 52.07 106.68)
+			(xy 189.23 143.51) (xy 189.23 139.7)
 		)
 		(stroke
@@
 	(wire
 		(pts
-			(xy 114.3 123.19) (xy 118.11 123.19)
+			(xy 175.26 55.88) (xy 177.8 55.88)
 		)
 		(stroke
@@
 	(wire
 		(pts
-			(xy 115.57 68.58) (xy 115.57 71.12)
+			(xy 50.8 106.68) (xy 52.07 106.68)
 		)
 		(stroke
@@
 	(wire
 		(pts
-			(xy 127 66.04) (xy 137.16 66.04)
+			(xy 114.3 123.19) (xy 118.11 123.19)
 		)
 		(stroke
@@
 	(wire
 		(pts
-			(xy 199.39 144.78) (xy 199.39 153.67)
+			(xy 115.57 68.58) (xy 115.57 71.12)
+		)
+		(stroke
+			(width 0)
+			(type default)
+		)
+	)
+	(wire
+		(pts
+			(xy 127 66.04) (xy 137.16 66.04)
 		)
 		(stroke
@@
 	(wire
 		(pts
+			(xy 213.36 146.05) (xy 203.2 146.05)
+		)
+		(stroke
+			(width 0)
+			(type default)
+		)
+	)
+	(wire
+		(pts
 			(xy 127 66.04) (xy 127 68.58)
 		)
@@
 	(wire
 		(pts
+			(xy 175.26 58.42) (xy 177.8 58.42)
+		)
+		(stroke
+			(width 0)
+			(type default)
+		)
+	)
+	(wire
+		(pts
+			(xy 203.2 144.78) (xy 199.39 144.78)
+		)
+		(stroke
+			(width 0)
+			(type default)
+		)
+	)
+	(wire
+		(pts
 			(xy 107.95 71.12) (xy 113.03 71.12)
 		)
@@
 	(wire
 		(pts
+			(xy 213.36 146.05) (xy 213.36 153.67)
+		)
+		(stroke
+			(width 0)
+			(type default)
+		)
+	)
+	(wire
+		(pts
 			(xy 113.03 140.97) (xy 118.11 140.97)
 		)
@@
 	(wire
 		(pts
-			(xy 128.27 101.6) (xy 128.27 102.87)
-		)
-		(stroke
-			(width 0)
-			(type default)
-		)
-	)
-	(wire
-		(pts
 			(xy 127 68.58) (xy 127 72.39)
 		)
@@
 	(wire
 		(pts
+			(xy 146.05 128.27) (xy 143.51 128.27)
+		)
+		(stroke
+			(width 0)
+			(type default)
+		)
+	)
+	(wire
+		(pts
 			(xy 107.95 57.15) (xy 107.95 71.12)
 		)
@@
 		)
 	)
+	(global_label "A0"
+		(shape input)
+		(at 146.05 128.27 0)
+		(fields_autoplaced yes)
+		(effects
+			(font
+				(size 1.27 1.27)
+			)
+			(justify left)
+		)
+		(property "Intersheetrefs" "${INTERSHEET_REFS}"
+			(at 151.3333 128.27 0)
+			(effects
+				(font
+					(size 1.27 1.27)
+				)
+				(justify left)
+				(hide yes)
+			)
+		)
+	)
 	(global_label "A5"
 		(shape input)
@@
 		)
 	)
+	(global_label "A0"
+		(shape input)
+		(at 175.26 58.42 180)
+		(fields_autoplaced yes)
+		(effects
+			(font
+				(size 1.27 1.27)
+			)
+			(justify right)
+		)
+		(property "Intersheetrefs" "${INTERSHEET_REFS}"
+			(at 169.9767 58.42 0)
+			(effects
+				(font
+					(size 1.27 1.27)
+				)
+				(justify right)
+				(hide yes)
+			)
+		)
+	)
 	(global_label "A4"
 		(shape input)
@@
 	)
 	(symbol
-		(lib_id "Connector:Conn_01x03_Socket")
-		(at 182.88 53.34 0)
-		(unit 1)
-		(exclude_from_sim no)
-		(in_bom yes)
-		(on_board yes)
-		(dnp no)
-		(property "Reference" "J4"
-			(at 184.15 52.0699 0)
-			(effects
-				(font
-					(size 1.27 1.27)
-				)
-				(justify left)
-			)
-		)
-		(property "Value" "Conn_01x03_Socket"
-			(at 170.434 60.198 0)
-			(effects
-				(font
-					(size 1.27 1.27)
-				)
-				(justify left)
-			)
-		)
-		(property "Footprint" "Connector_PinHeader_2.54mm:PinHeader_1x03_P2.54mm_Vertical"
-			(at 182.88 53.34 0)
-			(effects
-				(font
-					(size 1.27 1.27)
-				)
-				(hide yes)
-			)
-		)
-		(property "Datasheet" "~"
-			(at 182.88 53.34 0)
-			(effects
-				(font
-					(size 1.27 1.27)
-				)
-				(hide yes)
-			)
-		)
-		(property "Description" "Generic connector, single row, 01x03, script generated"
-			(at 182.88 53.34 0)
-			(effects
-				(font
-					(size 1.27 1.27)
-				)
-				(hide yes)
-			)
-		)
-		(pin "3"
-		)
-		(pin "1"
-		)
-		(pin "2"
-		)
-		(instances
-			(project ""
-				(path "/b28ec357-7924-445c-8320-f5bf00c8aa67"
-					(reference "J4")
-					(unit 1)
-				)
-			)
-		)
-	)
-	(symbol
 		(lib_id "Regulator_Linear:LM7805_TO220")
 		(at 127 57.15 0)
@@
 	)
 	(symbol
+		(lib_id "Connector:Conn_01x04_Socket")
+		(at 182.88 53.34 0)
+		(unit 1)
+		(exclude_from_sim no)
+		(in_bom yes)
+		(on_board yes)
+		(dnp no)
+		(fields_autoplaced yes)
+		(property "Reference" "J5"
+			(at 184.15 53.3399 0)
+			(effects
+				(font
+					(size 1.27 1.27)
+				)
+				(justify left)
+			)
+		)
+		(property "Value" "Conn_01x04_Socket"
+			(at 184.15 55.8799 0)
+			(effects
+				(font
+					(size 1.27 1.27)
+				)
+				(justify left)
+			)
+		)
+		(property "Footprint" "Connector_PinHeader_2.54mm:PinHeader_1x04_P2.54mm_Vertical"
+			(at 182.88 53.34 0)
+			(effects
+				(font
+					(size 1.27 1.27)
+				)
+				(hide yes)
+			)
+		)
+		(property "Datasheet" "~"
+			(at 182.88 53.34 0)
+			(effects
+				(font
+					(size 1.27 1.27)
+				)
+				(hide yes)
+			)
+		)
+		(property "Description" "Generic connector, single row, 01x04, script generated"
+			(at 182.88 53.34 0)
+			(effects
+				(font
+					(size 1.27 1.27)
+				)
+				(hide yes)
+			)
+		)
+		(pin "4"
+		)
+		(pin "3"
+		)
+		(pin "1"
+		)
+		(pin "2"
+		)
+		(instances
+			(project ""
+				(path "/b28ec357-7924-445c-8320-f5bf00c8aa67"
+					(reference "J5")
+					(unit 1)
+				)
+			)
+		)
+	)
+	(symbol
 		(lib_id "Device:R")
 		(at 64.77 148.59 0)
@@
 					(unit 1)
 				)
-			)
-		)
-	)
-	(symbol
-		(lib_id "power:+5V")
-		(at 128.27 101.6 0)
-		(unit 1)
-		(exclude_from_sim no)
-		(in_bom yes)
-		(on_board yes)
-		(dnp no)
-		(fields_autoplaced yes)
-		(property "Reference" "#PWR017"
-			(at 128.27 105.41 0)
-			(effects
-				(font
-					(size 1.27 1.27)
-				)
-				(hide yes)
-			)
-		)
-		(property "Value" "+5V"
-			(at 128.27 96.52 0)
-			(effects
-				(font
-					(size 1.27 1.27)
-				)
-			)
-		)
-		(property "Footprint" ""
-			(at 128.27 101.6 0)
-			(effects
-				(font
-					(size 1.27 1.27)
-				)
-				(hide yes)
-			)
-		)
-		(property "Datasheet" ""
-			(at 128.27 101.6 0)
-			(effects
-				(font
-					(size 1.27 1.27)
-				)
-				(hide yes)
-			)
-		)
-		(property "Description" "Power symbol creates a global label with name \"+5V\""
-			(at 128.27 101.6 0)
-			(effects
-				(font
-					(size 1.27 1.27)
-				)
-				(hide yes)
-			)
-		)
-		(pin "1"
-		)
-		(instances
-			(project "coil_winding"
-				(path "/b28ec357-7924-445c-8320-f5bf00c8aa67"
-					(reference "#PWR017")
-					(unit 1)
-				)
