File: Hardware/Pcb/coil_winding_v3/front_panel/front_panel.kicad_sch (KiCad schematic)
At the start: 17 parts, among them J1 Conn_01x14_Socket, J4 Conn_01x13_Socket, SW1 SW_Push, SW2 SW_Push, SW3 RotaryEncoder_Switch

Commit message: final_code
Parts:
- removed RV1: R_Potentiometer, Potentiometer_THT:Potentiometer_Runtron_RM-065_Vertical, symbol Device:R_Potentiometer
- removed SW1: SW_Push, Button_Switch_THT:SW_PUSH_6mm_H7.3mm, symbol Switch:SW_Push
Connections:
- net +3V3: now also J1.8 (Pin_8)
- net D2: now also J4.11 (Pin_11); no longer J4.10 (Pin_10)
- net D3: now also J4.10 (Pin_10); no longer J4.9 (Pin_9)
- net D4: now also J4.12 (Pin_12); no longer J4.11 (Pin_11)
- net D7: now also J4.9 (Pin_9); no longer J4.12 (Pin_12)
- net D8: no longer names the net of J4.13 (Pin_13)
